File: docs/kicad/laser_board/laser_board.kicad_pcb (KiCad board)
At the start: 2 copper layers, 24.1 x 41.9 mm, 4 parts, among them J1 Barrel_Jack_Switch, J2 Conn_01x03, J3 Conn_01x02, SW1 SW_SPDT

Commit message: docs - added Laser Board to laser page
Parts:
- added REF**: myMountingHole_3.2mm_M3, 0_my_footprints:myMountingHole_3.2mm_M3, F.Cu at (12.7, -3.81)
- added REF**: myMountingHole_3.2mm_M3, 0_my_footprints:myMountingHole_3.2mm_M3, F.Cu at (12.7, -38.1)
- J1: footprint cnc3018-PCB:myBarrelJack -> 0_my_footprints:myBarrelJack
- J2: footprint cnc3018-PCB:big_3pin -> 0_my_footprints:Phoenix5.08x3
- SW1: footprint cnc3018-PCB:SW_DPDT_BLUE_LEVER -> 0_my_footprints:mySwitchToggleSPDT
Routing:
- net Net-(J1-Pad2): vias 2 -> 0
Changed lines of the file:
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@@
     (thickness 1.6)
     (drawings 8)
-    (tracks 8)
+    (tracks 6)
     (zones 0)
-    (modules 4)
+    (modules 6)
     (nets 6)
   )
@@
     (add_net "Net-(J2-Pad2)")
   )
-  (module cnc3018-PCB:myBarrelJack (layer F.Cu)
+  (module 0_my_footprints:myMountingHole_3.2mm_M3 (layer F.Cu)
+    (at 12.7 -3.81)
+    (descr "Mounting Hole 3.2mm, no annular, M3")
+    (tags "mounting hole 3.2mm no annular m3")
+    (attr virtual)
+    (fp_text reference REF** (at 0 -4.2) (layer B.Fab)
+      (effects (font (size 1 1) (thickness 0.15)))
+    )
+    (fp_text value myMountingHole_3.2mm_M3 (at 0 4.2) (layer B.Fab)
+      (effects (font (size 1 1) (thickness 0.15)))
+    )
+    (fp_circle (center 0 0) (end 3.2 0) (layer F.SilkS) (width 0.15))
+    (pad "" np_thru_hole circle (at 0 0) (size 3.2 3.2) (drill 3.2) (layers *.Cu *.Mask))
+  )
+  (module 0_my_footprints:myMountingHole_3.2mm_M3 (layer F.Cu)
+    (at 12.7 -38.1)
+    (descr "Mounting Hole 3.2mm, no annular, M3")
+    (tags "mounting hole 3.2mm no annular m3")
+    (attr virtual)
+    (fp_text reference REF** (at 0 -4.2) (layer B.Fab)
+      (effects (font (size 1 1) (thickness 0.15)))
+    )
+    (fp_text value myMountingHole_3.2mm_M3 (at 0 4.2) (layer B.Fab)
+      (effects (font (size 1 1) (thickness 0.15)))
+    )
+    (fp_circle (center 0 0) (end 3.2 0) (layer F.SilkS) (width 0.15))
+    (pad "" np_thru_hole circle (at 0 0) (size 3.2 3.2) (drill 3.2) (layers *.Cu *.Mask))
+  )
+  (module 0_my_footprints:Phoenix5.08x3 (layer F.Cu)
+    (at 19.05 -12.7 270)
+    (fp_text reference J2 (at 0 -7.62 90) (layer F.SilkS)
+      (effects (font (size 1 1) (thickness 0.15)))
+    )
+    (fp_text value Conn_01x03 (at 0 -5.08 90) (layer F.Fab)
+      (effects (font (size 1 1) (thickness 0.15)))
+    )
+    (fp_line (start 7.62 2.54) (end -7.62 2.54) (layer F.SilkS) (width 0.12))
+    (fp_line (start 7.62 -2.54) (end 7.62 2.54) (layer F.SilkS) (width 0.12))
+    (fp_line (start -7.62 -2.54) (end 7.62 -2.54) (layer F.SilkS) (width 0.12))
+    (fp_line (start -7.62 -2.54) (end -7.62 2.54) (layer F.SilkS) (width 0.12))
+    (fp_line (start -7.62 2.54) (end -7.62 -8.89) (layer F.Fab) (width 0.12))
+    (fp_line (start -7.62 -8.89) (end 7.62 -8.89) (layer F.Fab) (width 0.12))
+    (fp_line (start 7.62 -8.89) (end 7.62 2.54) (layer F.Fab) (width 0.12))
+    (fp_line (start 7.62 2.54) (end -7.62 2.54) (layer F.Fab) (width 0.12))
+    (pad 3 thru_hole circle (at 5.08 0 270) (size 3 3) (drill 1.2) (layers *.Cu *.Mask)
+      (net 1 "Net-(J1-Pad2)"))
+    (pad 2 thru_hole circle (at 0 0 270) (size 3 3) (drill 1.2) (layers *.Cu *.Mask)
+      (net 5 "Net-(J2-Pad2)"))
+    (pad 1 thru_hole circle (at -5.08 0 270) (size 3 3) (drill 1.2) (layers *.Cu *.Mask)
+      (net 4 "Net-(J2-Pad1)"))
+    (model ${KISYS3DMOD}/Connector_Phoenix_MSTB.3dshapes/PhoenixContact_MSTBA_2,5_3-G-5,08_1x03_P5.08mm_Horizontal.wrl
+      (offset (xyz 5.08 0 0))
+      (scale (xyz 1 1 1))
+      (rotate (xyz 0 0 180))
+    )
+  )
+  (module 0_my_footprints:myBarrelJack (layer F.Cu)
     (at 15.24 -29.21 180)
     (descr "DC Barrel Jack")
@@
     )
     (fp_text value Barrel_Jack_Switch (at -6.2 -5.5) (layer F.Fab)
+      (effects (font (size 1 1) (thickness 0.15)))
+    )
+    (fp_text user %R (at -3 -2.95) (layer F.Fab)
       (effects (font (size 1 1) (thickness 0.15)))
     )
@@
     (fp_line (start 0.8 4.5) (end 0.8 -3.75) (layer F.Fab) (width 0.1))
     (fp_line (start 0 -4.5) (end -13.7 -4.5) (layer F.Fab) (width 0.1))
-    (fp_text user %R (at -3 -2.95) (layer F.Fab)
-      (effects (font (size 1 1) (thickness 0.15)))
-    )
-    (pad 2 thru_hole circle (at -6.096 -1.016 180) (size 2.2 2.2) (drill 1) (layers *.Cu *.Mask)
-      (net 1 "Net-(J1-Pad2)"))
-    (pad 2 thru_hole circle (at -6.096 0 180) (size 2.2 2.2) (drill 1) (layers *.Cu *.Mask)
-      (net 1 "Net-(J1-Pad2)"))
-    (pad 2 thru_hole circle (at -6.096 1.016 180) (size 2.2 2.2) (drill 1) (layers *.Cu *.Mask)
-      (net 1 "Net-(J1-Pad2)"))
-    (pad 1 thru_hole circle (at 0 -1.016 180) (size 2.2 2.2) (drill 1) (layers *.Cu *.Mask)
-      (net 2 "Net-(J1-Pad1)"))
-    (pad 1 thru_hole circle (at 0 0 180) (size 2.2 2.2) (drill 1) (layers *.Cu *.Mask)
-      (net 2 "Net-(J1-Pad1)"))
-    (pad 1 thru_hole circle (at 0 1.016 180) (size 2.2 2.2) (drill 1) (layers *.Cu *.Mask)
-      (net 2 "Net-(J1-Pad1)"))
-    (pad 3 thru_hole circle (at -4.064 4.826 180) (size 2.2 2.2) (drill 1) (layers *.Cu *.Mask)
+    (pad 3 thru_hole circle (at -2.032 4.826 180) (size 2.2 2.2) (drill 1) (layers *.Cu *.Mask)
       (net 3 "Net-(J1-Pad3)"))
     (pad 3 thru_hole circle (at -3.048 4.826 180) (size 2.2 2.2) (drill 1) (layers *.Cu *.Mask)
       (net 3 "Net-(J1-Pad3)"))
-    (pad 3 thru_hole circle (at -2.032 4.826 180) (size 2.2 2.2) (drill 1) (layers *.Cu *.Mask)
+    (pad 3 thru_hole circle (at -4.064 4.826 180) (size 2.2 2.2) (drill 1) (layers *.Cu *.Mask)
       (net 3 "Net-(J1-Pad3)"))
-    (model ${KISYS3DMOD}/Connector_BarrelJack.3dshapes/BarrelJack_Horizontal.wrl
-      (at (xyz 0 0 0))
+    (pad 1 thru_hole circle (at 0 1.016 180) (size 2.2 2.2) (drill 1) (layers *.Cu *.Mask)
+      (net 2 "Net-(J1-Pad1)"))
+    (pad 1 thru_hole circle (at 0 0 180) (size 2.2 2.2) (drill 1) (layers *.Cu *.Mask)
+      (net 2 "Net-(J1-Pad1)"))
+    (pad 1 thru_hole circle (at 0 -1.016 180) (size 2.2 2.2) (drill 1) (layers *.Cu *.Mask)
+      (net 2 "Net-(J1-Pad1)"))
+    (pad 2 thru_hole circle (at -6.096 1.016 180) (size 2.2 2.2) (drill 1) (layers *.Cu *.Mask)
+      (net 1 "Net-(J1-Pad2)"))
+    (pad 2 thru_hole circle (at -6.096 0 180) (size 2.2 2.2) (drill 1) (layers *.Cu *.Mask)
+      (net 1 "Net-(J1-Pad2)"))
+    (pad 2 thru_hole circle (at -6.096 -1.016 180) (size 2.2 2.2) (drill 1) (layers *.Cu *.Mask)
+      (net 1 "Net-(J1-Pad2)"))
+    (model C:/src/kiCad/libraries/my_3d_files/DC_PowerJack.step
+      (offset (xyz -7 0 0))
       (scale (xyz 1 1 1))
-      (rotate (xyz 0 0 0))
-    )
-  )
-  (module cnc3018-PCB:big_3pin (layer F.Cu)
-    (at 19.05 -12.7 270)
-    (fp_text reference J2 (at 0 -7.62 90) (layer F.SilkS)
-      (effects (font (size 1 1) (thickness 0.15)))
-    )
-    (fp_text value Conn_01x03 (at 0 -5.08 90) (layer F.Fab)
-      (effects (font (size 1 1) (thickness 0.15)))
-    )
-    (fp_line (start -7.62 -2.54) (end -7.62 2.54) (layer F.SilkS) (width 0.12))
-    (fp_line (start -7.62 -2.54) (end 7.62 -2.54) (layer F.SilkS) (width 0.12))
-    (fp_line (start 7.62 -2.54) (end 7.62 2.54) (layer F.SilkS) (width 0.12))
-    (fp_line (start 7.62 2.54) (end -7.62 2.54) (layer F.SilkS) (width 0.12))
-    (pad 1 thru_hole circle (at -5.08 0 270) (size 3 3) (drill 1.2) (layers *.Cu *.Mask)
-      (net 4 "Net-(J2-Pad1)"))
-    (pad 2 thru_hole circle (at 0 0 270) (size 3 3) (drill 1.2) (layers *.Cu *.Mask)
-      (net 5 "Net-(J2-Pad2)"))
-    (pad 3 thru_hole circle (at 5.08 0 270) (size 3 3) (drill 1.2) (layers *.Cu *.Mask)
-      (net 1 "Net-(J1-Pad2)"))
+      (rotate (xyz -90 0 90))
+    )
   )
   (module cnc3018-PCB:my2pin (layer F.Cu)
@@
       (effects (font (size 1 1) (thickness 0.15)))
     )
+    (fp_line (start 3.81 -1.27) (end 1.27 -1.27) (layer F.SilkS) (width 0.12))
+    (fp_line (start 3.81 1.27) (end 3.81 -1.27) (layer F.SilkS) (width 0.12))
+    (fp_line (start -1.27 1.27) (end 3.81 1.27) (layer F.SilkS) (width 0.12))
+    (fp_circle (center 0 0) (end 0 -1.27) (layer F.SilkS) (width 0.12))
+    (fp_line (start -1.27 -1.27) (end 1.27 -1.27) (layer F.SilkS) (width 0.12))
     (fp_line (start -1.27 -1.27) (end -1.27 1.27) (layer F.SilkS) (width 0.12))
-    (fp_line (start -1.27 -1.27) (end 1.27 -1.27) (layer F.SilkS) (width 0.12))
-    (fp_circle (center 0 0) (end 0 -1.27) (layer F.SilkS) (width 0.12))
-    (fp_line (start -1.27 1.27) (end 3.81 1.27) (layer F.SilkS) (width 0.12))
-    (fp_line (start 3.81 1.27) (end 3.81 -1.27) (layer F.SilkS) (width 0.12))
-    (fp_line (start 3.81 -1.27) (end 1.27 -1.27) (layer F.SilkS) (width 0.12))
     (pad 1 thru_hole circle (at 0 0 90) (size 2.2 2.2) (drill 0.8) (layers *.Cu *.Mask)
       (net 1 "Net-(J1-Pad2)"))
@@
       (net 5 "Net-(J2-Pad2)"))
   )
-  (module cnc3018-PCB:SW_DPDT_BLUE_LEVER (layer F.Cu)
+  (module 0_my_footprints:mySwitchToggleSPDT (layer F.Cu)
     (at 6.35 -27.94 270)
     (fp_text reference SW1 (at 0 5.08 90) (layer F.SilkS)
@@
     (pad 3 thru_hole circle (at 4.5 0 270) (size 2.2 2.2) (drill 1) (layers *.Cu *.Mask)
       (net 4 "Net-(J2-Pad1)"))
+    (model C:/src/kiCad/libraries/my_3d_files/switch_blue.step
+      (offset (xyz 0 0 10.2))
+      (scale (xyz 1 1 1))
+      (rotate (xyz 0 0 90))
+    )
   )
   (dimension 34.29 (width 0.15) (layer Dwgs.User)
@@
     (arrow2b (pts (xy 46.99 -41.91) (xy 47.576421 -40.783496)))
   )
-  (via (at 12.7 -38.1) (size 3.4) (drill 3.2) (layers F.Cu B.Cu) (net 1))
-  (via (at 12.7 -3.81) (size 3.4) (drill 3.2) (layers F.Cu B.Cu) (net 1))
   (segment (start 15.24 -28.194) (end 7.366 -28.194) (width 4) (layer B.Cu) (net 2))
   (segment (start 6.35 -29.21) (end 6.35 -32.44) (width 4) (layer B.Cu) (net 2))
